File: DigitalIO/DigitalIOTop/DigitalIO_3_3V_LevelShift.brd (EAGLE design)
At the start: 66.5 x 62.2 mm, 13 parts, among them K1 HF46105, K2 HF46105, K3 HF46105, K4 HF46105, Q1 691131710002, Q2 691131710002, Q3 691131710002, Q4 691131710002

Commit message: Increase drill from 2.5mm to 2.75mm. Remove not need holes.
Other:
- outline, holes or cut-outs redrawn
Changed lines of the file:
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@@
 <board>
 <plain>
-<wire x1="0" y1="0" x2="66.5" y2="0" width="0" layer="20"/>
+<wire x1="0" y1="0" x2="30.6" y2="0" width="0" layer="20"/>
+<wire x1="30.6" y1="0" x2="30.6" y2="1.5" width="0" layer="20"/>
+<wire x1="30.6" y1="1.5" x2="35.9" y2="1.5" width="0" layer="20"/>
+<wire x1="35.9" y1="1.5" x2="35.9" y2="0" width="0" layer="20"/>
+<wire x1="35.9" y1="0" x2="66.5" y2="0" width="0" layer="20"/>
 <wire x1="66.5" y1="0" x2="66.5" y2="62.2" width="0" layer="20"/>
-<wire x1="66.5" y1="62.2" x2="0" y2="62.2" width="0" layer="20"/>
+<wire x1="66.5" y1="62.2" x2="35.9" y2="62.2" width="0" layer="20"/>
+<wire x1="35.9" y1="62.2" x2="35.9" y2="60.7" width="0" layer="20"/>
+<wire x1="35.9" y1="60.7" x2="30.6" y2="60.7" width="0" layer="20"/>
+<wire x1="30.6" y1="60.7" x2="30.6" y2="62.2" width="0" layer="20"/>
+<wire x1="30.6" y1="62.2" x2="0" y2="62.2" width="0" layer="20"/>
 <wire x1="0" y1="62.2" x2="0" y2="0" width="0" layer="20"/>
-<hole x="8.25" y="49.2" drill="2.5"/>
-<hole x="58.25" y="13" drill="2.5"/>
+<hole x="8.25" y="49.2" drill="2.75"/>
+<hole x="58.25" y="13" drill="2.75"/>
 <text x="58.25" y="16.85" size="1.778" layer="16" font="vector" ratio="10" rot="MR180" align="center">8DI/8DO</text>
-<hole x="8.25" y="13" drill="2.5"/>
-<hole x="58.25" y="49.2" drill="2.5"/>
+<hole x="8.25" y="13" drill="2.75"/>
+<hole x="58.25" y="49.2" drill="2.75"/>
 <circle x="8.25" y="4.15" radius="1" width="1.6" layer="30"/>
 <circle x="13.25" y="4.15" radius="1" width="1.6" layer="30"/>
