File: DigitalIO/DigitalIOTop/DigitalIO.brd (EAGLE design)
At the start: 66.5 x 62.2 mm, 9 parts, among them K1 HF46105, K2 HF46105, K3 HF46105, K4 HF46105, Q1 691131710002, Q2 691131710002, Q3 691131710002, Q4 691131710002, X1 87438-06

Commit message: Rework to operate with 5V only. Add INT and RESET signals.
Signed-off-by: Alexander Falkenstern <alexander.falkenstern@gmail.com>
Parts:
- removed X1: 87438-06, con-molex:87438-06
- added P1: PH-06SMT, con-jst-ph:S6B-PH-SM4
- moved K1 0.15 mm to (20.2, 22.6)
- moved K2 0.15 mm to (28.8, 22.6)
- moved K3 0.15 mm to (37.8, 22.6)
- moved K4 0.15 mm to (46.2, 22.6)
Connections:
- net +5V: now also P1.1; no longer X1.1
- net GND: now also P1.6; no longer X1.6
- net N$14: now also P1.4; no longer X1.4
- net N$2: now also P1.3; no longer X1.3
- net N$4: now also P1.5; no longer X1.5
- net N$5: now also P1.2; no longer X1.2
Routing:
- net +5V: track 50.0 -> 43.7 mm
- net N$14: track 14.1 -> 10.8 mm, vias 0 -> 1
- net N$5: track 15.4 -> 12.6 mm, vias 0 -> 1
- net N$4: track 20.1 -> 17.3 mm, vias 0 -> 1
- net N$2: track 11.2 -> 8.48 mm, vias 0 -> 1
- net N$13: track 45.4 -> 44.6 mm
- removed copper zone on layer 1, net +5V
- removed copper zone on layer 16, net +5V
- removed copper zone on layer 1, net N$10
- removed copper zone on layer 16, net N$10
- removed copper zone on layer 1, net N$11
- removed copper zone on layer 16, net N$11
- removed copper zone on layer 1, net N$12
- removed copper zone on layer 16, net N$12
- removed copper zone on layer 1, net N$13
- removed copper zone on layer 16, net N$13
- removed copper zone on layer 1, net N$14
- removed copper zone on layer 16, net N$14
- removed copper zone on layer 1, net N$2
- removed copper zone on layer 16, net N$2
- removed copper zone on layer 1, net N$4
- removed copper zone on layer 16, net N$4
- removed copper zone on layer 1, net N$5
- removed copper zone on layer 16, net N$5
- removed copper zone on layer 1, net N$6
- removed copper zone on layer 16, net N$6
- removed copper zone on layer 1, net N$7
- removed copper zone on layer 16, net N$7
- removed copper zone on layer 1, net N$8
- removed copper zone on layer 16, net N$8
- removed copper zone on layer 1, net N$9
- removed copper zone on layer 16, net N$9
