File: MainBoard/MainBoard.sch (EAGLE design)
At the start: 47 parts, among them IC1 3.3V, P1 DF11-06-2DS, Q1 BC337-40, Q2 BSS138, Q3 BSS138, Q4 BS170, Q5 BS170

Commit message: Replace On/Off fan with PWM driven one
Parts:
- removed D4: 1N4148, diode:1N4148DO35-2V
- added R20: 680R, rcl:R-EU_0204/2V
- F1: value 1.5A -> 1.35A; device ptc:PPTCPTH11MM -> ptc:PPTCRGEF250
- FAN: value 22-23-2031 -> 22-23-2041; device con-molex:22-23-2031 -> con-molex:22-23-2041
- Q1: value BC337-40 -> BS170; device transistor-npn:BC337-40 -> transistor-small-signal:BS170
- R10, R4: device rcl:R-EU_0204/2V -> rcl:R-EU_0204/5
- R11: value 10K -> 100R; device rcl:R-EU_0204/2V -> rcl:R-EU_0204/5
- R12: value 10K -> 1K
- R13: value 10K -> 1K; device rcl:R-EU_0204/2V -> rcl:R-EU_0204/5
- R14: value 10K -> 200R
- R15, R16: value 100R -> 1K8; device rcl:R-EU_0204/5 -> rcl:R-EU_0204/2V
- R17: value 100R -> 200R
- R18: value 100R -> 10K
- R19: value 680R -> 10K
- R3: value 10K -> 150R
- R5: value 10K -> 1K8
- R6: value 10K -> 1K2
- R7: value 1K -> 10K; device rcl:R-EU_0204/5 -> rcl:R-EU_0204/2V
- R8: value 1K -> 100R; device rcl:R-EU_0204/2V -> rcl:R-EU_0204/5
- R9: device rcl:R-EU_0204/5 -> rcl:R-EU_0204/2V
Connections:
- removed net 3V3: R1.2, R11.2, R13.2, R15.2, R16.2, R17.2, R18.2, R2.2, R5.1, R6.1, R7.2, R9.2, RPI.3V3
- removed net N$11: Q1.B, R3.2, R4.2
- removed net N$14: D4.A, FAN-3.S, Q1.C
- new net N$2: Q1.G, R3.1
- new net N$29: FAN-1.S, Q1.D, R4.2
- new net VCC: 433MHZ.VCC, 868MHZ.VCC, C1.1, C2.1, C3.1, IC1.OUT, R1.2, R2.2
- net +3V3: now also R10.2, R11.2, R13.2, R14.2, R16.2, R17.2, R19.2, R3.2, R5.2, R6.1, R7.1, R8.2, RPI.3V3; no longer 433MHZ.VCC, 868MHZ.VCC, C1.1, C2.1, C3.1, IC1.OUT
- net +5V: now also FAN-3.S, R15.1, R18.1, R4.1, R9.1; no longer D4.C, FAN-2.S, R10.1, R14.1, R8.1
- net GND: now also FAN-4.S; no longer Q1.E, R3.1
- net INT: now also R16.1; no longer R11.1
- net N$1: now also R12.2; no longer R10.2
- net N$12: now also R9.2; no longer R8.2
- net N$13: now also Q1.S, R5.1; no longer R4.1
- net N$21: now also R7.2; no longer R6.2
- net N$22: now also FAN-2.S, R6.2; no longer FAN-1.S, R5.2
- net N$23: now also R8.1; no longer R15.1
- net N$24: now also R11.1; no longer R16.1
- net N$25: now also R15.2; no longer R12.2
- net N$26: now also R18.2; no longer R14.2
- net N$27: now also R17.1; no longer R18.1
- net N$28: now also R14.1; no longer R17.1
- net N$5: now also R20.2; no longer R19.2
- net RESET: now also R20.1; no longer R13.1
- net SCL: now also R13.1; no longer R9.1
- net SDA: now also R10.1; no longer R7.1
Other:
- note removed: "+Fan"
- note removed: "-Fan"
- moved on the sheet: 24V, D1, D2, D3, F1, F2, F3, FAN-1, FAN-2, FAN-3, MP1584, MP2482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
